Commit message: quasi

File: launch/erc_joint_limited_robot.urdf.xacro (robot description, xacro)
@@ -22,5 +22,5 @@
     <parent link="world" />
     <child link = "base_link" />
-    <origin xyz="0.0 -0.052 -0.438" rpy="0.0 0.0 0.0" />
+    <origin xyz="0.0 -0.052 -0.42" rpy="0.0 0.0 1.570796 " />
   </joint>
   <!-- z value of joint same as height of robot base plane

File: launch/erc_robot.urdf.xacro (robot description, xacro)
@@ -11,10 +11,12 @@
     transmission_hw_interface="$(arg transmission_hw_interface)"
   />
-  <!--link name="world" /-->
-  <joint name="world_joint" type="fixed">
-    <!--parent link="world" /-->
-    <parent link="environment_0" />
+  <!-- constraints-->
+  <link name="world" />
+  <joint name="base_link_fix_location" type="fixed">
+    <parent link="world" />
     <child link = "base_link" />
-    <origin xyz="0.0 0.0 0.0" rpy="0.0 0.0 0.0" />
+    <origin xyz="0.0 -0.052 -0.42" rpy="0.0 0.0 1.570796 " />
   </joint>
+  <!-- z value of joint same as height of robot base plane
+	y value range: [-0.056 -0.048]=[farest closest] to the panel   -->
 </robot>
