Commit message: robot correct positioning and reference frame

File: launch/UR3_joint_limited_robot.urdf.xacro (robot description, xacro)
@@ -2,9 +2,17 @@
 <robot xmlns:xacro="http://wiki.ros.org/xacro"
        name="ur3" >
+  <!-- mechanical transmission parameters -->
   <xacro:arg name="transmission_hw_interface" default="hardware_interface/PositionJointInterface"/>
+  <!-- robot positioning parameters -->
+  <xacro:arg name="joint_x" default="0"/>
+  <xacro:arg name="joint_y" default="-0.052"/>
+  <xacro:arg name="joint_z" default="0.001"/>
+  <xacro:arg name="joint_R" default="0"/>
+  <xacro:arg name="joint_P" default="0"/>
+  <xacro:arg name="joint_Y" default="1.570796"/>
   <!-- common stuff -->
   <xacro:include filename="$(find ur_description)/urdf/common.gazebo.xacro" />
   <!-- ur3 macro inclusion-->
-  <xacro:include filename="$(find almasim)/launch/erc.urdf.xacro" />
+  <xacro:include filename="$(find almasim)/launch/UR3_assembler.urdf.xacro" />
   <!-- arm spawn-->
   <xacro:ur3_robot prefix="" joint_limited="true"
@@ -22,7 +30,10 @@
     <parent link="world" />
     <child link = "base_link" />
-    <origin xyz="0.0 -0.052 -0.42" rpy="0.0 0.0 1.570796 " />
+    <origin xyz="0.0 -0.052 0.001" rpy="0.0 0.0 1.570796 " />
+    <!--origin xyz="${arg joint_x} ${arg joint_y} ${arg joint_z}"
+ 	    rpy="${arg joint_R} ${arg joint_P} ${arg joint_Y}" /-->
   </joint>
-  <!-- z value of joint same as height of robot base plane
+  <!-- difference z-0.16 to avoid collision with box underneath-->
+  <!-- z value: minimal gap to avoid collision with robot joint base
 	y value range: [-0.056 -0.048]=[farest closest] to the panel   -->
 </robot>

File: launch/UR3_robot.urdf.xacro (robot description, xacro)
@@ -2,9 +2,17 @@
 <robot xmlns:xacro="http://wiki.ros.org/xacro"
        name="ur3" >
+  <!-- mechanical transmission parameters -->
   <xacro:arg name="transmission_hw_interface" default="hardware_interface/PositionJointInterface"/>
+  <!-- robot positioning parameters -->
+  <xacro:arg name="joint_x" default="0"/>
+  <xacro:arg name="joint_y" default="0"/>
+  <xacro:arg name="joint_z" default="0"/>
+  <xacro:arg name="joint_R" default="0"/>
+  <xacro:arg name="joint_P" default="0"/>
+  <xacro:arg name="joint_Y" default="0"/>
   <!-- common stuff -->
   <xacro:include filename="$(find ur_description)/urdf/common.gazebo.xacro" />
   <!-- ur3 macro inclusion -->
-  <xacro:include filename="$(find almasim)/launch/erc.urdf.xacro" />
+  <xacro:include filename="$(find almasim)/launch/UR3_assembler.urdf.xacro" />
   <!-- arm spawn-->
   <xacro:ur3_robot prefix="" joint_limited="false"

File: launch/UR3_robot_TEST.urdf.xacro (robot description, xacro)
@@ -2,13 +2,20 @@
 <robot xmlns:xacro="http://wiki.ros.org/xacro"
        name="ur3" >
+  <!-- robot mechanical parameters -->
+  <xacro:arg name="limited" default="false"/>
   <xacro:arg name="transmission_hw_interface" default="hardware_interface/PositionJointInterface"/>
-  <xacro:arg name="limited" default="false"/>
+  <!-- robot positioning parameters -->
+  <xacro:arg name="joint_x" default="0"/>
+  <xacro:arg name="joint_y" default="0"/>
+  <xacro:arg name="joint_z" default="0"/>
+  <xacro:arg name="joint_R" default="0"/>
+  <xacro:arg name="joint_P" default="0"/>
   <!-- common stuff -->
   <xacro:include filename="$(find ur_description)/urdf/common.gazebo.xacro" />
   <!-- ur3 macro inclusion -->
-  <xacro:include filename="$(find almasim)/launch/erc.urdf.xacro" />
+  <xacro:include filename="$(find almasim)/launch/UR3_assembly.urdf.xacro" />
   <!-- ARM SPAWN-->
   <!--limited joint motion-->
-  <xacro: if value="$(limited=='true')">
+  <xacro: if value="$(limited)">
 	  <xacro:ur3_robot prefix="" joint_limited="true"
 	    shoulder_pan_lower_limit="${-pi}" shoulder_pan_upper_limit="${pi}"
@@ -22,5 +29,5 @@
   <xacro:if/>
   <!-- unlimited joint motion-->
-  <xacro:unless value="$(limited=='true')">
+  <xacro:unless value="$(limited)">
 	  <xacro:ur3_robot prefix="" joint_limited="false"
 	    transmission_hw_interface="$(arg transmission_hw_interface)"

Commit message: launchers improvement

File: launch/UR3_joint_limited_robot.urdf.xacro (robot description, xacro)
@@ -4,11 +4,18 @@
   <!-- mechanical transmission parameters -->
   <xacro:arg name="transmission_hw_interface" default="hardware_interface/PositionJointInterface"/>
-  <!-- robot positioning parameters -->
-  <xacro:arg name="joint_x" default="0"/>
-  <xacro:arg name="joint_y" default="-0.052"/>
-  <xacro:arg name="joint_z" default="0.001"/>
-  <xacro:arg name="joint_R" default="0"/>
-  <xacro:arg name="joint_P" default="0"/>
-  <xacro:arg name="joint_Y" default="1.570796"/>
+  <xacro:arg name="limited" default="true"/>
+  <!-- robot positioning constraint parameters -->
+  <xacro:arg name="fix_joint_x" default="0"/>
+  <xacro:arg name="fix_joint_y" default="-0.052"/>
+  <xacro:arg name="fix_joint_z" default="0.001"/>
+  <xacro:arg name="fix_joint_R" default="0.0"/>
+  <xacro:arg name="fix_joint_P" default="0.0"/>
+  <xacro:arg name="fix_joint_Y" default="1.570796"/>
+  <!-- z:  to avoid collision with box underneath-->
+  <!-- z value: minimal gap to avoid collision with robot joint base
+	y value range: [-0.056 -0.048]=[farest closest] to the panel   -->
+  <!-- TODO verify wich REFSYS moveit is using: if there is discrepancy
+	wrt to the spawn one and the one with varied y here
+	TODO-->
   <!-- common stuff -->
   <xacro:include filename="$(find ur_description)/urdf/common.gazebo.xacro" />
@@ -30,10 +37,6 @@
     <parent link="world" />
     <child link = "base_link" />
-    <origin xyz="0.0 -0.052 0.001" rpy="0.0 0.0 1.570796 " />
-    <!--origin xyz="${arg joint_x} ${arg joint_y} ${arg joint_z}"
- 	    rpy="${arg joint_R} ${arg joint_P} ${arg joint_Y}" /-->
+    <origin xyz="$(arg fix_joint_x) $(arg fix_joint_y) $(arg fix_joint_z)"
+ 	    rpy="$(arg fix_joint_R) $(arg fix_joint_P) $(arg fix_joint_Y)" />
   </joint>
-  <!-- difference z-0.16 to avoid collision with box underneath-->
-  <!-- z value: minimal gap to avoid collision with robot joint base
-	y value range: [-0.056 -0.048]=[farest closest] to the panel   -->
 </robot>

File: launch/UR3_robot.urdf.xacro (robot description, xacro)
@@ -4,11 +4,18 @@
   <!-- mechanical transmission parameters -->
   <xacro:arg name="transmission_hw_interface" default="hardware_interface/PositionJointInterface"/>
-  <!-- robot positioning parameters -->
-  <xacro:arg name="joint_x" default="0"/>
-  <xacro:arg name="joint_y" default="0"/>
-  <xacro:arg name="joint_z" default="0"/>
-  <xacro:arg name="joint_R" default="0"/>
-  <xacro:arg name="joint_P" default="0"/>
-  <xacro:arg name="joint_Y" default="0"/>
+  <xacro:arg name="limited" default="true"/>
+  <!-- robot positioning constraint parameters -->
+  <xacro:arg name="fix_joint_x" default="0"/>
+  <xacro:arg name="fix_joint_y" default="-0.052"/>
+  <xacro:arg name="fix_joint_z" default="0.001"/>
+  <xacro:arg name="fix_joint_R" default="0.0"/>
+  <xacro:arg name="fix_joint_P" default="0.0"/>
+  <xacro:arg name="fix_joint_Y" default="1.570796"/>
+  <!-- z:  to avoid collision with box underneath-->
+  <!-- z value: minimal gap to avoid collision with robot joint base
+	y value range: [-0.056 -0.048]=[farest closest] to the panel   -->
+  <!-- TODO verify wich REFSYS moveit is using: if there is discrepancy
+	wrt to the spawn one and the one with varied y here
+	TODO-->
   <!-- common stuff -->
   <xacro:include filename="$(find ur_description)/urdf/common.gazebo.xacro" />
@@ -24,7 +31,6 @@
     <parent link="world" />
     <child link = "base_link" />
-    <origin xyz="0.0 -0.052 -0.42" rpy="0.0 0.0 1.570796 " />
+    <origin xyz="$(arg fix_joint_x) $(arg fix_joint_y) $(arg fix_joint_z)"
+ 	    rpy="$(arg fix_joint_R) $(arg fix_joint_P) $(arg fix_joint_Y)" />
   </joint>
-  <!-- z value of joint same as height of robot base plane
-	y value range: [-0.056 -0.048]=[farest closest] to the panel   -->
 </robot>

File: launch/UR3_robot_TEST.urdf.xacro (robot description, xacro)
@@ -3,20 +3,28 @@
        name="ur3" >
   <!-- robot mechanical parameters -->
-  <xacro:arg name="limited" default="false"/>
+  <xacro:property name="joint_limited" default="true"/>
   <xacro:arg name="transmission_hw_interface" default="hardware_interface/PositionJointInterface"/>
-  <!-- robot positioning parameters -->
-  <xacro:arg name="joint_x" default="0"/>
-  <xacro:arg name="joint_y" default="0"/>
-  <xacro:arg name="joint_z" default="0"/>
-  <xacro:arg name="joint_R" default="0"/>
-  <xacro:arg name="joint_P" default="0"/>
+  <!-- robot positioning constraint parameters -->
+  <xacro:arg name="fix_joint_x" default="0"/>
+  <xacro:arg name="fix_joint_y" default="-0.052"/>
+  <xacro:arg name="fix_joint_z" default="0.001"/>
+  <xacro:arg name="fix_joint_R" default="0.0"/>
+  <xacro:arg name="fix_joint_P" default="0.0"/>
+  <xacro:arg name="fix_joint_Y" default="1.570796"/>
+  <!-- z:  to avoid collision with box underneath-->
+  <!-- z value: minimal gap to avoid collision with robot joint base
+	y value range: [-0.056 -0.048]=[farest closest] to the panel   -->
+  <!-- TODO verify wich REFSYS moveit is using: if there is discrepancy
+	wrt to the spawn one and the one with varied y here
+	TODO-->
   <!-- common stuff -->
   <xacro:include filename="$(find ur_description)/urdf/common.gazebo.xacro" />
   <!-- ur3 macro inclusion -->
-  <xacro:include filename="$(find almasim)/launch/UR3_assembly.urdf.xacro" />
+  <xacro:include filename="$(find almasim)/launch/UR3_assembler.urdf.xacro" />
   <!-- ARM SPAWN-->
   <!--limited joint motion-->
-  <xacro: if value="$(limited)">
-	  <xacro:ur3_robot prefix="" joint_limited="true"
+  <!--xacro: if value="${limited=='true'}"-->
+  <xacro: if value="${joint_limited}">
+	  <xacro:ur3_robot prefix="" joint_limited="$(arg joint_limited)"
 	    shoulder_pan_lower_limit="${-pi}" shoulder_pan_upper_limit="${pi}"
 	    shoulder_lift_lower_limit="${-pi}" shoulder_lift_upper_limit="${pi}"
@@ -27,11 +35,11 @@
 	    transmission_hw_interface="$(arg transmission_hw_interface)"
 	  />
-  <xacro:if/>
+  </xacro:if>
   <!-- unlimited joint motion-->
-  <xacro:unless value="$(limited)">
-	  <xacro:ur3_robot prefix="" joint_limited="false"
+  <!--xacro:unless value="${limited=='true'}">
+	  <xacro:ur3_robot prefix="" joint_limited="$(arg limited)"
 	    transmission_hw_interface="$(arg transmission_hw_interface)"
 	  />
-  <xacro:unless/>
+  </xacro:unless-->
   <!-- constraints-->
   <link name="world" />
@@ -39,8 +47,6 @@
     <parent link="world" />
     <child link = "base_link" />
-    <origin xyz="0.0 -0.052 0.161" rpy="0.0 0.0 1.570796" />
-    <!--origin xyz="0.0 -0.052 -0.438" rpy="0.0 0.0 0.0" /-->
+    <origin xyz="$(arg fix_joint_x) $(arg fix_joint_y) $(arg fix_joint_z)"
+ 	    rpy="$(arg fix_joint_R) $(arg fix_joint_P) $(arg fix_joint_Y)" />
   </joint>
-  <!-- z value of joint same as height of robot base plane
-	y value range: [-0.056 -0.048]=[farest closest] to the panel   -->
 </robot>
